Commit message: Update turtlebot3_waffle_pi.urdf.xacro
remove camera to speed up simulation

File: turtlebot3/turtlebot3_description/urdf/turtlebot3_waffle_pi.urdf.xacro (robot description, xacro)
@@ -160,5 +160,5 @@
     </inertial>
   </link>
-  <joint name="camera_joint" type="fixed">
+<!--   <joint name="camera_joint" type="fixed">
     <origin xyz="0.073 -0.011 0.084" rpy="0 0 0"/>
     <parent link="base_link"/>
@@ -184,4 +184,4 @@
     <child link="camera_rgb_optical_frame"/>
   </joint>
-  <link name="camera_rgb_optical_frame"/>
+  <link name="camera_rgb_optical_frame"/> -->
 </robot>
